File: modules/lamp_module/lamp_module.kicad_sch (KiCad schematic)
At the start: 34 parts, among them J1 Screw_Terminal_01x02, J2 Screw_Terminal_01x02, J3 Conn_01x06_Socket, K1 12V 5A, K2 12V 5A, Q1 2N7002H, Q2 2N7002H, U1 ESP-12E, U3 AMS1117-3.3, U4 PC817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

Commit message: Lamp module PCB V1.0 finished
Parts:
- added D5: LED, LED_SMD:LED_0603_1608Metric, symbol Device:LED
- added R11: 2.2k, Resistor_SMD:R_0603_1608Metric, symbol Device:R
- C4: renamed from C5; footprint Capacitor_SMD:C_0201_0603Metric -> Capacitor_SMD:C_0603_1608Metric
- D1: renamed from D2; footprint Diode_THT:D_DO-35_SOD27_P7.62mm_Horizontal -> Diode_SMD:D_SOD-323F
- D2: renamed from D1; footprint Diode_THT:D_DO-35_SOD27_P7.62mm_Horizontal -> Diode_SMD:D_SOD-323F
- J3: footprint Connector_PinHeader_1.27mm:PinHeader_1x06_P1.27mm_Vertical -> Connector_PinHeader_2.54mm:PinHeader_1x06_P2.54mm_Vertical
- R1: renamed from R10; footprint Resistor_SMD:R_0201_0603Metric -> Resistor_SMD:R_0603_1608Metric
- R10: renamed from R6; footprint Resistor_SMD:R_0201_0603Metric -> Resistor_SMD:R_0603_1608Metric
- R2: renamed from R9; footprint Resistor_SMD:R_0201_0603Metric -> Resistor_SMD:R_0603_1608Metric
- R3: renamed from R8; footprint Resistor_SMD:R_0201_0603Metric -> Resistor_SMD:R_0603_1608Metric
- R4: renamed from R7; footprint Resistor_SMD:R_0201_0603Metric -> Resistor_SMD:R_0603_1608Metric
- R5: renamed from R1; footprint Resistor_SMD:R_0201_0603Metric -> Resistor_SMD:R_0603_1608Metric; Power 1/4W -> 1/10W
- R6: renamed from R3; footprint Resistor_SMD:R_0201_0603Metric -> Resistor_SMD:R_0603_1608Metric; Power 1/4W -> 1/10W
- R7: renamed from R2; footprint Resistor_SMD:R_0201_0603Metric -> Resistor_SMD:R_0603_1608Metric
- R8: renamed from R4; footprint Resistor_SMD:R_0201_0603Metric -> Resistor_SMD:R_0603_1608Metric
- R9: renamed from R5; footprint (none) -> Resistor_THT:R_Axial_DIN0309_L9.0mm_D3.2mm_P12.70mm_Horizontal; Power (none) -> 2W; Tolerance (none) -> 5%
- U4, U5, U6: footprint Package_DIP:DIP-4_W7.62mm -> Package_DIP:SMDIP-4_W7.62mm
- renumbered C4 to C3, C7 to C5, D4 to D3, D5 to D4, U3 to U1, U1 to U2
Connections:
- net +12V: now also R11.2
- net GND: now also D5.1 (K)
- net SWITCH_NO: now also J2.1 (Pin_1); no longer J2.2 (Pin_2)
- net SWITCH_C: no longer names the net of K2.12
- net SWITCH_C: now also J2.2 (Pin_2); no longer J2.1 (Pin_1)
- new net: D5.2 (A), R11.1
Other:
- note added: "12V TO 3.3V REGULATION"
- note added: "LAMP FEEDBACK"
- note added: "POWER LED"
- note added: "RELAYS CONTROL"
- note added: "SERIAL CONNECTOR"
- note added: "WIFI MODULE"
- note removed: "O circuito é alimentado em 220V, pela rede elétrica da casa. Essa tensão é retificada e rebaixada para 3,3V. A tensão regulada é utilizada para alimentar todo o restante do circuito. O relé é controlado pelo módulo ESP-12E através de uma saída digital."
- company: (none) -> Alan Carvalho
- title: (none) -> Lamp Module
- moved on the sheet: C1, C2, C3, C4, C5, C6, D1, D2, D3, D4, F1, J1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
