File: modules/lamp_module/lamp_module.kicad_pcb (KiCad board)
At the start: 2 copper layers, 61 x 64 mm, 40 parts, among them J1 Screw_Terminal_01x02, J2 Screw_Terminal_01x02, J3 Conn_01x06_Socket, K1 12V 5A, K2 12V 5A, Q1 2N7002H, Q2 2N7002H, U1 AMS1117-3.3, U2 ESP-12E, U4 PC817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

Commit message: Lamp module 3D model finished
Other:
- board text added: "Designed by Alan Carvalho"
- board text added: "HV"
- board text added: "LV"
- board text added: "Lamp Module X1 V1.0"
Changed lines of the file:
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@@
   (gr_arc (start 122.11575 132.85025) (mid 119.994429 131.971571) (end 119.11575 129.85025)
     (stroke (width 0.2) (type default)) (layer "Edge.Cuts"))
+  (gr_text "LV" (at 133.604 107.442) (layer "B.SilkS")
+    (effects (font (size 2.5 2.5) (thickness 0.4) bold) (justify mirror))
+  )
+  (gr_text "Lamp Module X1 V1.0" (at 146.812 87.122 270) (layer "B.SilkS")
+    (effects (font (size 2 2) (thickness 0.4) bold) (justify mirror))
+  )
+  (gr_text "HV" (at 166.37 107.442) (layer "B.SilkS")
+    (effects (font (size 2.5 2.5) (thickness 0.4) bold) (justify mirror))
+  )
+  (gr_text "Designed by Alan Carvalho" (at 142.748 103.886 270) (layer "B.SilkS")
+    (effects (font (size 1.5 1.5) (thickness 0.3) bold) (justify left bottom mirror))
+  )
   (gr_text "L" (at 178.47875 77.04525) (layer "F.SilkS")
     (effects (font (size 1 1) (thickness 0.15)))
@@
     )
   )
+  (group "" (id 9f2d2d15-199d-41f6-9405-f09bc78ef925)
+    (members
+      343b3c6a-0f4b-448c-9bfc-fa16453c7aca
+      f63cba1e-f023-4d82-9dab-4d92edcfa6e4
+    )
+  )
