File: modules/lamp_module_x1/PCB/lamp_module_x1.kicad_pcb (KiCad board)
At the start: 2 copper layers, 48 x 63 mm, 29 parts, among them J1 Screw_Terminal_01x02, J2 Screw_Terminal_01x03, J3 Conn_01x06_Socket, J4 Conn_01x03_Socket, K1 12V 5A, Q1 2N7002H, U1 AMS1117-3.3, U2 ESP-12E, U4 PC817

Commit message: Switch feedback implemented
Connections:
- J2 pad 2: SWITCH_NO -> SWITCH
- J2 pad 3: SWITCH_C -> GND
- U2 pad 6: SWITCH_C -> SWITCH
- U2 pad 7: SWITCH_NO -> unconnected-(U2-GPIO13-Pad7)
Routing:
- net SWITCH_C: track 50.8 -> 0.00 mm, vias 1 -> 0
- net SWITCH: track 0.00 -> 46.0 mm, vias 0 -> 1
- net SWITCH_NO: track 44.6 -> 0.00 mm, vias 1 -> 0

Commit message: Lamp module X1 PCB finished
Parts:
- removed F1: 0.5A, Fuse:Fuse_0603_1608Metric
- added SW1: SW_SPDT, MyLibrary:Toggle_Switch_SelfLocking_7x7, F.Cu at (171.7, 61.0)
- moved J1 2.06 mm to (164.1, 58.1)
- moved J2 2.06 mm to (150.9, 58.1)
- moved G*** 0.53 mm to (154.4, 74.6)
Routing:
- net Net-(J1-Pin_2): track 37.0 -> 14.6 mm
- net LINE: track 36.2 -> 55.0 mm
- net GND: track 21.7 -> 19.4 mm, vias 9 -> 8
- net NEUT: track 19.6 -> 20.4 mm
- net SWITCH: track 46.0 -> 46.9 mm
- net LAMP: track 42.9 -> 43.7 mm

Commit message: Fabrication files updated
Parts:
- moved J3 12.7 mm to (132.1, 93.0), turned to 0 degrees
- renumbered R4 to R3, R5 to R4, R6 to R5, R7 to R6, U4 to U3
Routing:
- net RX: track 24.1 -> 14.3 mm
- net TX: track 18.5 -> 14.8 mm
- net +3.3V: track 74.9 -> 72.7 mm
Other:
- board text added: "JLCJLCJLCJLC"
