File: modules/on_off_module_x2/PCB/on_off_module_x2.kicad_pcb (KiCad board)
At the start: 2 copper layers, 63 x 63 mm, 38 parts, among them J1 Screw_Terminal_01x02, J2 Conn_01x06_Socket, J3 Conn_01x03_Socket, J4 Screw_Terminal_01x02, J5 Screw_Terminal_01x02, J6 Screw_Terminal_01x02, J7 Screw_Terminal_01x02, K1 12V 5A, K2 12V 5A, Q1 2N7002H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

Commit message: PCB gerber updated
Parts:
- moved G*** 18.7 mm to (157.6, 89.7)
Changed lines of the file:
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@@
         (effects (font (size 1 1) (thickness 0.15)))
     )
-    (fp_text user "L" (at 5.850238 6.096 unlocked) (layer "F.SilkS")
-        (effects (font (size 1 1) (thickness 0.15)))
-    )
-    (fp_text user "N" (at -0.65119 6.096 unlocked) (layer "F.SilkS")
+    (fp_text user "L" (at 5.850238 5.842 unlocked) (layer "F.SilkS")
+        (effects (font (size 1 1) (thickness 0.15)))
+    )
+    (fp_text user "N" (at -0.65119 5.842 unlocked) (layer "F.SilkS")
         (effects (font (size 1 1) (thickness 0.15)))
     )
@@
   )
   (footprint "LOGO" (layer "B.Cu")
-    (at 157.6832 71.047754 180)
+    (at 157.5816 89.7128 180)
     (attr board_only exclude_from_pos_files exclude_from_bom)
     (fp_text reference "G***" (at 0 0) (layer "B.SilkS") hide
@@
   (gr_arc (start 180.0912 119.481907) (mid 179.212531 121.603222) (end 177.0912 122.481907)
     (stroke (width 0.2) (type default)) (layer "Edge.Cuts"))
-  (gr_text "LV" (at 146.7612 76.381754) (layer "B.SilkS")
+  (gr_text "LV" (at 146.6596 95.0468) (layer "B.SilkS")
     (effects (font (size 2.5 2.5) (thickness 0.4) bold) (justify mirror))
   )
@@
     (effects (font (size 1.5 1.5) (thickness 0.3) bold) (justify mirror))
   )
-  (gr_text "HV" (at 157.6832 76.381754) (layer "B.SilkS")
+  (gr_text "HV" (at 157.5816 95.0468) (layer "B.SilkS")
     (effects (font (size 2.5 2.5) (thickness 0.4) bold) (justify mirror))
   )
