File: modules/sensor_module/PCB/sensor_module_x1.kicad_pcb (KiCad board)
At the start: 2 copper layers, 48 x 63 mm, 5 parts

Commit message: Sensor module PCB layout started
Parts:
- added BZ1: Buzzer, Buzzer_Beeper:Buzzer_12x9.5RM7.6, F.Cu at (-63.4, 111.2)
- added C1: 0.1uF, Capacitor_THT:C_Rect_L18.0mm_W6.0mm_P15.00mm_FKS3_FKP3, F.Cu at (82.9, 276.4)
- added C10: 10nF, Capacitor_SMD:C_0603_1608Metric, F.Cu at (55.4, 263.0)
- added C11: 10nF, Capacitor_SMD:C_0603_1608Metric, F.Cu at (47.6, 258.0)
- added C12: 10nF, Capacitor_SMD:C_0603_1608Metric, F.Cu at (43.8, 258.0)
- added C13: 10uF, Capacitor_SMD:CP_Elec_5x5.4, F.Cu at (46.4, 250.8)
- added C14: 47uF, Capacitor_SMD:CP_Elec_5x5.4, F.Cu at (39.4, 250.8)
- added C15: 10nF, Capacitor_SMD:C_0603_1608Metric, F.Cu at (49.5, 270.5)
- added C16: 10nF, Capacitor_SMD:C_0603_1608Metric, F.Cu at (45.8, 270.5)
- added C2: 100uF, Capacitor_SMD:CP_Elec_6.3x7.7, F.Cu at (-100.5, 122.2)
- added C3: 10uF, Capacitor_Tantalum_SMD:CP_EIA-3216-18_Kemet-A, F.Cu at (130.9, 144.8)
- added C4: 10uF, Capacitor_Tantalum_SMD:CP_EIA-3216-18_Kemet-A, F.Cu at (127.9, 144.7)
- added C5: 10uF, Capacitor_Tantalum_SMD:CP_EIA-3216-18_Kemet-A, F.Cu at (139.8, 144.8)
- added C6: 10uF, Capacitor_Tantalum_SMD:CP_EIA-3216-18_Kemet-A, F.Cu at (136.8, 144.8)
- added C7: 0.1uF, Capacitor_SMD:C_0603_1608Metric, F.Cu at (178.2, 103.5)
- added C8: 100nF, Capacitor_SMD:C_0603_1608Metric, F.Cu at (55.4, 248.1)
- added C9: 100nF, Capacitor_SMD:C_0603_1608Metric, F.Cu at (55.4, 244.3)
- added D1: GREEN, LED_SMD:LED_0603_1608Metric, F.Cu at (-50.0, 85.2)
- added D2: RED, LED_SMD:LED_0603_1608Metric, F.Cu at (-50.0, 87.7)
- added D3: BLUE, LED_SMD:LED_0603_1608Metric, F.Cu at (-50.0, 90.3)
- added D4: BLUE, LED_SMD:LED_0603_1608Metric, F.Cu at (-50.0, 92.9)
- added D5: BLUE, LED_SMD:LED_0603_1608Metric, F.Cu at (-50.0, 95.5)
- added J1: Screw_Terminal_01x02, TerminalBlock_Phoenix:TerminalBlock_Phoenix_MKDS-1,5-2-5.08_1x02_P5.08mm_Horizontal, F.Cu at (86.7, 116.2)
- added J2: Conn_01x06_Socket, Connector_PinHeader_2.54mm:PinHeader_1x06_P2.54mm_Vertical, F.Cu at (-76.5, 64.6)
- added J3: Conn_01x03_Socket, Connector_PinSocket_2.54mm:PinSocket_1x03_P2.54mm_Vertical, F.Cu at (-50.5, 106.7)
- added LDR1: 100k, OptoDevice:R_LDR_5.1x4.3mm_P3.4mm_Vertical, F.Cu at (159.8, 98.4)
- added POT1: 10k, Potentiometer_THT:Potentiometer_Bourns_3296W_Vertical, F.Cu at (-85.4, 86.6)
- added POT2: 10k, Potentiometer_THT:Potentiometer_Bourns_3296W_Vertical, F.Cu at (-85.4, 94.3)
- added POT3: 10k, Potentiometer_THT:Potentiometer_Bourns_3296W_Vertical, F.Cu at (-85.4, 102.0)
- added POT4: 10k, Potentiometer_THT:Potentiometer_Bourns_3296W_Vertical, F.Cu at (-85.4, 109.7)
- added PS1: HLK-PM12, Converter_ACDC:Converter_ACDC_HiLink_HLK-PMxx, F.Cu at (133.3, 99.7)
- added R1: 10k, Resistor_SMD:R_0603_1608Metric, F.Cu at (186.6, 103.5)
- added R10: 2k2, Resistor_SMD:R_0603_1608Metric, F.Cu at (52.1, 246.2)
- added R11: 10k, Resistor_SMD:R_0603_1608Metric, F.Cu at (61.0, 274.6)
- added R12: 47k, Resistor_SMD:R_0603_1608Metric, F.Cu at (55.3, 264.9)
- added R13: 1M, Resistor_SMD:R_0603_1608Metric, F.Cu at (47.6, 259.9)
- added R14: 2M, Resistor_SMD:R_0603_1608Metric, F.Cu at (43.8, 259.9)
- added R15: 10k, Resistor_SMD:R_0603_1608Metric, F.Cu at (47.6, 256.1)
- added R16: 47k, Resistor_SMD:R_0603_1608Metric, F.Cu at (43.8, 256.1)
- added R17: 1M, Resistor_SMD:R_0603_1608Metric, F.Cu at (51.6, 260.4)
- added R18: 1k, Resistor_SMD:R_0603_1608Metric, F.Cu at (-68.4, 108.2)
- added R19: 1k, Resistor_SMD:R_0603_1608Metric, F.Cu at (-68.4, 110.7)
- added R2: 10k, Resistor_SMD:R_0603_1608Metric, F.Cu at (190.6, 103.5)
- added R20: 1k, Resistor_SMD:R_0603_1608Metric, F.Cu at (-68.4, 113.2)
- added R3: 10k, Resistor_SMD:R_0603_1608Metric, F.Cu at (178.6, 125.1)
- added R4: 3k9, Resistor_SMD:R_0603_1608Metric, F.Cu at (-76.4, 113.2)
- added R5: 3k9, Resistor_SMD:R_0603_1608Metric, F.Cu at (-76.4, 115.7)
- added R6: 33k, Resistor_SMD:R_0603_1608Metric, F.Cu at (78.7, 259.1)
- added R7: 5k1, Resistor_SMD:R_0603_1608Metric, F.Cu at (77.4, 250.8)
- added R8: 47k, Resistor_SMD:R_0603_1608Metric, F.Cu at (55.4, 246.2)
- added R9: 1k2, Resistor_SMD:R_0603_1608Metric, F.Cu at (52.1, 244.3)
- added SW1: SW_SPDT, MyLibrary:Toggle_Switch_SelfLocking_7x7, F.Cu at (84.9, 285.2)
- added U1: AMS1117-3.3, Package_TO_SOT_SMD:SOT-223-3_TabPin2, F.Cu at (128.3, 137.2)
- added U2: AMS1117-5, Package_TO_SOT_SMD:SOT-223-3_TabPin2, F.Cu at (137.2, 137.2)
- added U3: ESP-12E, ESP8266:ESP-12E_SMD, F.Cu at (191.4, 107.3)
- added U4: LM393, Package_SO:SOIC-8-1EP_3.9x4.9mm_P1.27mm_EP2.62x3.51mm, F.Cu at (78.7, 263.1)
- added U5: MQ-5, Sensor:MQ-6, F.Cu at (149.0, 110.9)
- added U6: LM393, Package_SO:SOIC-8-1EP_3.9x4.9mm_P1.27mm_EP2.62x3.51mm, F.Cu at (52.1, 240.0)
- added U7: DHT11, MyLibrary:SNR4-2.54-15.5X12.0X5.5MM, F.Cu at (152.4, 133.3)
- added U8: PIR, MyLibrary:TO5, F.Cu at (148.0, 98.4)
- added U9: BISS0001, MyLibrary:SOIC127P600X180-16N, F.Cu at (47.6, 265.6)
- moved G*** 114.5 mm to (347.1, 64.7)
- moved REF** 114.5 mm to (324.9, 44.0)
- moved REF** 114.5 mm to (366.9, 101.0)
- moved REF** 114.5 mm to (324.9, 101.0)
- moved REF** 114.5 mm to (366.9, 44.0)
